Commit message: add HARIMOTO

File: src/HARIMOTO/urdf/HARIMOTO.urdf (robot description, URDF)
Before this commit: robot HARIMOTO, 5 links, 4 joints
Links:
- removed link arm
- removed link hand
- added link lower_arm, mass 0.0477129093267453; collision mesh filename=package://HARIMOTO/meshes/lower_arm.STL; visual mesh filename=package://HARIMOTO/meshes/lower_arm.STL
- added link upper_arm, mass 0.0214573443165031; collision mesh filename=package://HARIMOTO/meshes/upper_arm.STL; visual mesh filename=package://HARIMOTO/meshes/upper_arm.STL
- link base_link: mass 0.0151156528348089 -> 0.0468580060932661
- link lower_shoulder: mass 0.0335476434855063 -> 0.0576719241727568
- link upper_shoulder: mass 0.0317423532584571 -> 0.0335476434855063
Joints:
- removed joint arm
- removed joint hand
- removed joint uppler_shoulder
- added joint lower_arm: type revolute, parent upper_arm, child lower_arm, origin xyz=0.1085 0.0166 0.0151 rpy=0 0 3.1416, axis 0 0 -1, limit lower=-1.5 upper=1.5 effort=0 velocity=10
- added joint upper_arm: type revolute, parent lower_shoulder, child upper_arm, origin xyz=-0.0275 -0.124 0 rpy=-1.5708 0 -1.5708, axis 0 -1 0, limit lower=-0.7 upper=0.7 effort=0 velocity=10
- added joint upper_shoulder: type revolute, parent base_link, child upper_shoulder, origin xyz=0.27658 -0.037897 0.095074 rpy=0.18413 0.71623 2.0474, axis 0 0 1, limit lower=-1.2 upper=0 effort=0 velocity=10
- joint lower_shoulder: axis 1 0 0 -> 0 1 0; limit lower=-2.35 upper=0.785 effort=0 velocity=10 -> lower=-2.7 upper=0.75 effort=0 velocity=10; origin xyz=-0.018453 -0.010996 0 rpy=-3.1416 0 -0.38339 -> xyz=-0.005 -0.0145 -0.041 rpy=1.5708 -1.5708 0

Commit message: add HARIMOTO

File: src/HARIMOTO/urdf/HARIMOTO.urdf (robot description, URDF)
Before this commit: robot HARIMOTO, 5 links, 4 joints
Links:
- added link hand, mass 0.0425234840552025; collision mesh filename=package://HARIMOTO/meshes/hand.STL; visual mesh filename=package://HARIMOTO/meshes/hand.STL
- link lower_arm: mass 0.0477129093267453 -> 0.00518942527154281
- link lower_shoulder: mass 0.0576719241727568 -> 0.0576719241727569
Joints:
- added joint hand: type fixed, parent lower_arm, child hand, origin xyz=0 0 0 rpy=0 0 0, axis 0 0 0

Commit message: succeeded in running sample drive code!

File: src/HARIMOTO/urdf/HARIMOTO.urdf (robot description, URDF)
Before this commit: robot HARIMOTO, 6 links, 5 joints
Joints:
- joint hand: origin xyz=0 0 0 rpy=0 0 0 -> xyz=-0.11 0 0 rpy=0 0 0
- joint lower_arm: origin xyz=0.1085 0.0166 0.0151 rpy=0 0 3.1416 -> xyz=0 0 -0.02 rpy=0 0 3.1416
- joint lower_shoulder: origin xyz=-0.005 -0.0145 -0.041 rpy=1.5708 -1.5708 0 -> xyz=0.033 -0.0145 -0.041 rpy=-2.35 -1.5708 0
- joint upper_arm: origin xyz=-0.0275 -0.124 0 rpy=-1.5708 0 -1.5708 -> xyz=0 -0.1 0 rpy=-1.5708 0 -1.5708
- joint upper_shoulder: limit lower=-1.2 upper=0 effort=0 velocity=10 -> lower=-1 upper=0 effort=0 velocity=10; origin xyz=0.27658 -0.037897 0.095074 rpy=0.18413 0.71623 2.0474 -> xyz=0 0 0.3 rpy=-1.57 -1.57 0

Commit message: update minimal.launch

File: src/HARIMOTO/urdf/HARIMOTO.urdf (robot description, URDF)
Before this commit: robot HARIMOTO, 6 links, 5 joints
Links:
- added link front_left_wheel_link, mass 0.095024; collision cylinder length=0.02 radius=0.03; visual mesh filename=package://HARIMOTO/meshes/front_left_wheel_link.dae
- added link front_right_wheel_link, mass 0.095024; collision cylinder length=0.02 radius=0.03; visual mesh filename=package://HARIMOTO/meshes/front_right_wheel_link.dae
- added link rear_left_wheel_link, mass 0.095024; collision cylinder length=0.02 radius=0.03; visual mesh filename=package://HARIMOTO/meshes/rear_left_wheel_link.dae
- added link rear_right_wheel_link, mass 0.095024; collision cylinder length=0.02 radius=0.03; visual mesh filename=package://HARIMOTO/meshes/rear_right_wheel_link.dae
Joints:
- added joint front_left_wheel_joint: type continuous, parent base_link, child front_left_wheel_link, origin xyz=0.0505 -0.097 0.0435 rpy=0.0 -0.0 0.0, axis 1. 0. 0., limit effort=100 velocity=6.55
- added joint front_right_wheel_joint: type continuous, parent base_link, child front_right_wheel_link, origin xyz=-0.0505 -0.097 0.0435 rpy=0.0 -0.0 0.0, axis 1. 0. 0., limit effort=100 velocity=6.55
- added joint rear_left_wheel_joint: type continuous, parent base_link, child rear_left_wheel_link, origin xyz=0.0505 -0.097 -0.0435 rpy=0.0 -0.0 0.0, axis 1. 0. 0., limit effort=100 velocity=6.55
- added joint rear_right_wheel_joint: type continuous, parent base_link, child rear_right_wheel_link, origin xyz=-0.0505 -0.097 -0.0435 rpy=0.0 -0.0 0.0, axis 1. 0. 0., limit effort=100 velocity=6.55

Commit message: update HARIMOTO.urdf, correct wheel info, add camera_link!

File: src/HARIMOTO/urdf/HARIMOTO.urdf (robot description, URDF)
Before this commit: robot HARIMOTO, 10 links, 9 joints
Links:
- added link camera_link, mass 0.1; collision box size=0.025 0.09 0.025; visual box size=0.025 0.09 0.025
- link base_link: geometry collision box size=0.2 0.2 0.3; visual box size=0.04 0.1 0.14
Joints:
- added joint camera_joint: type fixed, parent base_link, child camera_link, origin xyz=0 0.05 0.25 rpy=0 0 0
- joint front_left_wheel_joint: origin xyz=0.0505 -0.097 0.0435 rpy=0.0 -0.0 0.0 -> xyz=0 0.13 0.16 rpy=0.0 -0.0 1.5708
- joint front_right_wheel_joint: axis 1. 0. 0. -> -1. 0. 0.; origin xyz=-0.0505 -0.097 0.0435 rpy=0.0 -0.0 0.0 -> xyz=0 -0.03 0.16 rpy=0.0 -0.0 1.5708
- joint rear_left_wheel_joint: origin xyz=0.0505 -0.097 -0.0435 rpy=0.0 -0.0 0.0 -> xyz=-0.17 0.13 0.16 rpy=0.0 -0.0 1.5708
- joint rear_right_wheel_joint: axis 1. 0. 0. -> -1. 0. 0.; origin xyz=-0.0505 -0.097 -0.0435 rpy=0.0 -0.0 0.0 -> xyz=-0.17 -0.03 0.16 rpy=0.0 -0.0 1.5708
